File: boards/shield/v1/v1.kicad_pcb (KiCad board)
At the start: 4 copper layers, 120 x 67.5 mm, 138 parts, among them J1 Pickup, J10 Conn_01x02, J11 Conn_01x02, J12 Conn_02x06_Top_Bottom, J2 Output jack, J3 USB_B_Micro, J4 SWD, J5 oled, J6 Conn_01x02, J7 Conn_01x02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

Commit message: code folder
Parts:
- removed R5: 22k, Resistor_SMD:R_0603_1608Metric
- removed R6: 10k, Resistor_SMD:R_0603_1608Metric
- C36: value 10.6nF -> 10n
- C38: value 2.05n -> 2n
- C43: footprint Capacitor_SMD:C_0603_1608Metric -> Capacitor_SMD:C_1210_3225Metric
- C5: value 10u -> 47u; footprint Capacitor_SMD:C_0603_1608Metric -> Capacitor_SMD:C_1210_3225Metric
- D1, D2: footprint Diode_SMD:D_0603_1608Metric_Pad1.05x0.95mm_HandSolder -> Diode_SMD:D_0603_1608Metric
- R34: value 6.34k -> 6.8k
- R37: value 8.66k -> 8.2k
- U10: footprint Package_SO:TSSOP-16_4.4x5mm_P0.65mm -> JFHADC:PW16
- U11, U8: footprint Package_SO:MSOP-8_3x3mm_P0.65mm -> JFHAnalog:OPA1602AIDR
- moved D2 4.20 mm to (94.5, 106.0), turned to 90 degrees
- moved D1 3.90 mm to (94.5, 110.0), turned to -90 degrees
- moved U11 3.59 mm to (189.3, 94.1), turned to -90 degrees
- moved U8 3.20 mm to (189.3, 82.6), turned to -90 degrees
- moved C31 2.30 mm to (178.3, 121.1)
- moved C32 2.30 mm to (178.3, 119.2)
- moved C5 2.15 mm to (199.3, 83.5)
- moved C38 1.58 mm to (184.0, 80.0)
- moved R37 1.58 mm to (184.0, 82.0)
- moved C39 1.51 mm to (194.1, 78.0)
- moved C43 0.61 mm to (198.6, 96.1)
- moved C44 0.50 mm to (184.0, 93.5)
- moved R3 0.50 mm to (184.0, 87.5)
- moved R34 0.50 mm to (184.0, 95.5)
- moved R39 0.50 mm to (184.0, 89.5)
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Connections:
- D1 pad 1: /USB_DN -> /USB_DP
- D2 pad 1: /USB_DP -> /USB_DN
- U8 pad 6: Net-(R5-Pad2) -> Net-(C5-Pad1)
- U8 pad 7: Net-(R5-Pad2) -> Net-(C5-Pad1)
Routing:
- net /ADC/SIG_IN_ADC: track 64.0 -> 54.1 mm
- net Net-(R34-Pad1): track 7.23 -> 14.3 mm, vias 0 -> 2
- net /DAC/S_OUT: track 45.8 -> 38.9 mm, vias 0 -> 2
- net Net-(R39-Pad2): track 13.3 -> 8.46 mm, vias 2 -> 0
- net Net-(C43-Pad2): track 9.01 -> 13.5 mm
- net Net-(R5-Pad2): track 3.99 -> 0.00 mm
- net Net-(C40-Pad2): track 23.3 -> 20.8 mm
- net Net-(R39-Pad1): track 11.4 -> 13.2 mm
- net GNDA: track 0.00 -> 1.52 mm, vias 17 -> 19
- net Net-(C38-Pad1): track 17.6 -> 19.0 mm, vias 2 -> 0
- net Net-(C36-Pad1): track 13.1 -> 14.3 mm
- net +3.3VA: track 13.2 -> 14.4 mm, vias 14 -> 13
- net /SIG_OUT: track 21.8 -> 20.7 mm
- net /input_filter/SIG_IN1: track 3.65 -> 2.88 mm
