File: boards/shield/v1/v1.kicad_sch (KiCad schematic)
At the start: 46 parts, among them J1 Pickup, J2 Output jack, SW3 SW_DPDT_x2, U1 HT75xx-1-SOT89, U2 GND_STARPOINT, U3 RP2040, U6 TCR2EF33, U7 REF3433

Commit message: code folder
Other:
- moved on the sheet: U2
